File: hw/sch_pcb/4XLTO1865V01A.kicad_pcb (KiCad board)
At the start: 2 copper layers, 60.5 x 49.7 mm, 7 parts, among them J1 HEADER_2x04_PARALLEL, J2 HEADER_2x04_PARALLEL, J3 HEADER_2x04_PARALLEL

Commit message: Edit PCB
Other:
- board text added: "4XLTO1865V01A JACHO"
- board text added: "MLAB.CZ 2022"
Changed lines of the file:
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@@
   (gr_arc (start 114.554 77.602) (mid 117.482932 70.530932) (end 124.554 67.602) (layer "Edge.Cuts") (width 0.1))
   (gr_line (start 114.554 117.348) (end 175.006 117.348) (layer "Edge.Cuts") (width 0.1))
+  (gr_text "MLAB.CZ\n2022" (at 120.142 92.202 90) (layer "F.SilkS")
+    (effects (font (size 1.5 1.5) (thickness 0.3)))
+  )
+  (gr_text "4XLTO1865V01A\nJACHO" (at 169.926 91.948 90) (layer "F.SilkS")
+    (effects (font (size 1.5 1.5) (thickness 0.3)))
+  )
   (segment (start 146.05 113.102) (end 146.05 110.582) (width 0.5) (layer "F.Cu") (net 1))
   (segment (start 146.05 110.582) (end 152.53 104.102) (width 0.5) (layer "F.Cu") (net 1))

Commit message: Edit PCB
Routing:
- net GND: vias 0 -> 16
Changed lines of the file:
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@@
     )
   )
+  (gr_rect (start 164.211 114.554) (end 175.133 117.348) (layer "B.Mask") (width 0.15) (fill solid))
+  (gr_rect (start 114.427 114.554) (end 125.349 117.348) (layer "B.Mask") (width 0.15) (fill solid))
   (gr_line (start 124.554 67.602) (end 165.006 67.602) (layer "Edge.Cuts") (width 0.1))
   (gr_line (start 175.006 117.348) (end 175.006 77.602) (layer "Edge.Cuts") (width 0.1))
@@
   (segment (start 152.308 108.042) (end 152.4 107.95) (width 0.5) (layer "B.Cu") (net 2))
   (segment (start 140.97 108.042) (end 152.308 108.042) (width 0.5) (layer "B.Cu") (net 2))
+  (via (at 120.904 115.57) (size 0.9) (drill 0.5) (layers "F.Cu" "B.Cu") (free) (net 3))
+  (via (at 117.094 115.57) (size 0.9) (drill 0.5) (layers "F.Cu" "B.Cu") (free) (net 3))
+  (via (at 115.824 115.57) (size 0.9) (drill 0.5) (layers "F.Cu" "B.Cu") (free) (net 3))
+  (via (at 171.196 115.57) (size 0.9) (drill 0.5) (layers "F.Cu" "B.Cu") (free) (net 3))
+  (via (at 124.714 115.57) (size 0.9) (drill 0.5) (layers "F.Cu" "B.Cu") (free) (net 3))
+  (via (at 173.736 115.57) (size 0.9) (drill 0.5) (layers "F.Cu" "B.Cu") (free) (net 3))
+  (via (at 172.466 115.57) (size 0.9) (drill 0.5) (layers "F.Cu" "B.Cu") (free) (net 3))
+  (via (at 118.364 115.57) (size 0.9) (drill 0.5) (layers "F.Cu" "B.Cu") (free) (net 3))
+  (via (at 119.634 115.57) (size 0.9) (drill 0.5) (layers "F.Cu" "B.Cu") (free) (net 3))
+  (via (at 166.116 115.57) (size 0.9) (drill 0.5) (layers "F.Cu" "B.Cu") (free) (net 3))
+  (via (at 168.656 115.57) (size 0.9) (drill 0.5) (layers "F.Cu" "B.Cu") (free) (net 3))
+  (via (at 164.846 115.57) (size 0.9) (drill 0.5) (layers "F.Cu" "B.Cu") (free) (net 3))
+  (via (at 169.926 115.57) (size 0.9) (drill 0.5) (layers "F.Cu" "B.Cu") (free) (net 3))
+  (via (at 123.444 115.57) (size 0.9) (drill 0.5) (layers "F.Cu" "B.Cu") (free) (net 3))
+  (via (at 167.386 115.57) (size 0.9) (drill 0.5) (layers "F.Cu" "B.Cu") (free) (net 3))
+  (via (at 122.174 115.57) (size 0.9) (drill 0.5) (layers "F.Cu" "B.Cu") (free) (net 3))
   (zone (net 3) (net_name "GND") (layers F&B.Cu) (hatch edge 0.508)
-    (connect_pads yes (clearance 0.508))
+    (connect_pads yes (clearance 0.2))
     (min_thickness 0.254) (filled_areas_thickness no)
     (fill yes (thermal_gap 0.508) (thermal_bridge_width 0.508))
@@
       )
     )
+  )
+  (zone (net 3) (net_name "GND") (layer "B.Cu") (hatch edge 0.508)
+    (connect_pads yes (clearance 0.01))
+    (min_thickness 0.254) (filled_areas_thickness no)
+    (fill yes (thermal_gap 0.508) (thermal_bridge_width 0.508))
+    (polygon
+      (pts
+        (xy 178.816 122.174)
+        (xy 108.966 124.968)
+        (xy 108.712 113.284)
+        (xy 178.562 113.284)
+      )
+    )

Commit message: Edit PCB
Parts:
- added M1: HOLE, Mlab_Mechanical:MountingHole_3mm, F.Cu at (119.4, 92.5)
- added M2: HOLE, Mlab_Mechanical:MountingHole_3mm, F.Cu at (170.2, 92.5)
- added R1: 10K NTC, Resistor_SMD:R_0805_2012Metric_Pad1.20x1.40mm_HandSolder, F.Cu at (144.8, 92.5)
Connections:
- J2 pad 2: GND -> Net-(J2-Pad2)
- J2 pad 3: GND -> Net-(J2-Pad3)
Routing:
- net Net-(J2-Pad3): track 0.00 -> 40.4 mm, vias 0 -> 1
- net Net-(J2-Pad2): track 0.00 -> 37.4 mm, vias 0 -> 1
Changed lines of the file:
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@@
   (net 2 "/Battery-")
   (net 3 "GND")
+  (net 4 "Net-(J2-Pad2)")
+  (net 5 "Net-(J2-Pad3)")
   (footprint "Mlab_Pin_Headers:Angled_1x04" (layer "F.Cu")
     (at 144.78 113.102 -90)
@@
       (net 3 "GND") (pintype "input"))
     (pad "2" thru_hole rect (at 0 -1.27 270) (size 1.524 1.524) (drill 0.889) (layers *.Cu *.Mask "F.SilkS")
-      (net 3 "GND") (pintype "input"))
+      (net 4 "Net-(J2-Pad2)") (pintype "input"))
     (pad "3" thru_hole rect (at 0 1.27 270) (size 1.524 1.524) (drill 0.889) (layers *.Cu *.Mask "F.SilkS")
-      (net 3 "GND") (pintype "input"))
+      (net 5 "Net-(J2-Pad3)") (pintype "input"))
     (pad "4" thru_hole rect (at 0 3.81 270) (size 1.524 1.524) (drill 0.889) (layers *.Cu *.Mask "F.SilkS")
       (net 3 "GND") (pintype "input"))
     (model "${KICAD6_3DMODEL_DIR}/Connector_PinHeader_2.54mm.3dshapes/PinHeader_1x04_P2.54mm_Horizontal.wrl"
       (offset (xyz 0 3.81 0))
+      (scale (xyz 1 1 1))
+      (rotate (xyz 0 0 0))
+    )
+  )
+  (footprint "Mlab_Mechanical:MountingHole_3mm" placed (layer "F.Cu")
+    (at 119.38 92.475)
+    (descr "Mounting hole, Befestigungsbohrung, 3mm, No Annular, Kein Restring,")
+    (tags "Mounting hole, Befestigungsbohrung, 3mm, No Annular, Kein Restring,")
+    (property "Sheetfile" "4XLTO1865V01A.kicad_sch")
+    (property "Sheetname" "")
+    (attr through_hole)
+    (fp_text reference "M1" (at 0 -4.191) (layer "F.SilkS") hide
+      (effects (font (size 1.524 1.524) (thickness 0.3048)))
+    )
+    (fp_text value "HOLE" (at 0 4.191) (layer "F.SilkS") hide
+      (effects (font (size 1.524 1.524) (thickness 0.3048)))
+    )
+    (fp_circle (center 0 0) (end 2.99974 0) (layer "F.Fab") (width 0.381) (fill none))
+    (pad "1" thru_hole circle (at 0 0) (size 6 6) (drill 3) (layers *.Cu *.Mask)
+      (net 3 "GND") (pintype "input") (clearance 1) (zone_connect 2))
+    (model "${MLAB}/src/3d/mechanical/m3_komplet.step"
+      (offset (xyz 0 0 0))
       (scale (xyz 1 1 1))
       (rotate (xyz 0 0 0))
@@
     )
   )
+  (footprint "Resistor_SMD:R_0805_2012Metric_Pad1.20x1.40mm_HandSolder" (layer "F.Cu")
+    (at 144.78 92.475 -90)
+    (descr "Resistor SMD 0805 (2012 Metric), square (rectangular) end terminal, IPC_7351 nominal with elongated pad for handsoldering. (Body size source: IPC-SM-782 page 72, https://www.pcb-3d.com/wordpress/wp-content/uploads/ipc-sm-782a_amendment_1_and_2.pdf), generated with kicad-footprint-generator")
+    (tags "resistor handsolder")
+    (property "Sheetfile" "4XLTO1865V01A.kicad_sch")
+    (property "Sheetname" "")
+    (attr smd)
+    (fp_text reference "R1" (at 0 -1.65 90) (layer "F.SilkS")
+      (effects (font (size 1 1) (thickness 0.15)))
+    )
+    (fp_text value "10K NTC" (at 0 1.65 90) (layer "F.Fab")
+      (effects (font (size 1 1) (thickness 0.15)))
+    )
+    (fp_text user "${REFERENCE}" (at 0 0 90) (layer "F.Fab")
+      (effects (font (size 0.5 0.5) (thickness 0.08)))
+    )
+    (fp_line (start -0.227064 -0.735) (end 0.227064 -0.735) (layer "F.SilkS") (width 0.12))
+    (fp_line (start -0.227064 0.735) (end 0.227064 0.735) (layer "F.SilkS") (width 0.12))
+    (fp_line (start -1.85 0.95) (end -1.85 -0.95) (layer "F.CrtYd") (width 0.05))
+    (fp_line (start 1.85 -0.95) (end 1.85 0.95) (layer "F.CrtYd") (width 0.05))
+    (fp_line (start 1.85 0.95) (end -1.85 0.95) (layer "F.CrtYd") (width 0.05))
+    (fp_line (start -1.85 -0.95) (end 1.85 -0.95) (layer "F.CrtYd") (width 0.05))
+    (fp_line (start -1 -0.625) (end 1 -0.625) (layer "F.Fab") (width 0.1))
+    (fp_line (start 1 -0.625) (end 1 0.625) (layer "F.Fab") (width 0.1))
+    (fp_line (start 1 0.625) (end -1 0.625) (layer "F.Fab") (width 0.1))
+    (fp_line (start -1 0.625) (end -1 -0.625) (layer "F.Fab") (width 0.1))
+    (pad "1" smd roundrect (at -1 0 270) (size 1.2 1.4) (layers "F.Cu" "F.Paste" "F.Mask") (roundrect_rratio 0.208333)
+      (net 5 "Net-(J2-Pad3)") (pintype "passive"))
+    (pad "2" smd roundrect (at 1 0 270) (size 1.2 1.4) (layers "F.Cu" "F.Paste" "F.Mask") (roundrect_rratio 0.208333)
+      (net 4 "Net-(J2-Pad2)") (pintype "passive"))
+    (model "${KICAD6_3DMODEL_DIR}/Resistor_SMD.3dshapes/R_0805_2012Metric.wrl"
+      (offset (xyz 0 0 0))
+      (scale (xyz 1 1 1))
+      (rotate (xyz 0 0 0))
+    )
+  )
+  (footprint "Mlab_Mechanical:MountingHole_3mm" placed (layer "F.Cu")
+    (at 170.18 92.475)
+    (descr "Mounting hole, Befestigungsbohrung, 3mm, No Annular, Kein Restring,")
+    (tags "Mounting hole, Befestigungsbohrung, 3mm, No Annular, Kein Restring,")
+    (property "Sheetfile" "4XLTO1865V01A.kicad_sch")
+    (property "Sheetname" "")
+    (attr through_hole)
+    (fp_text reference "M2" (at 0 -4.191) (layer "F.SilkS") hide
+      (effects (font (size 1.524 1.524) (thickness 0.3048)))
+    )
+    (fp_text value "HOLE" (at 0 4.191) (layer "F.SilkS") hide
+      (effects (font (size 1.524 1.524) (thickness 0.3048)))
+    )
+    (fp_circle (center 0 0) (end 2.99974 0) (layer "F.Fab") (width 0.381) (fill none))
+    (pad "1" thru_hole circle (at 0 0) (size 6 6) (drill 3) (layers *.Cu *.Mask)
+      (net 3 "GND") (pintype "input") (clearance 1) (zone_connect 2))
+    (model "${MLAB}/src/3d/mechanical/m3_komplet.step"
+      (offset (xyz 0 0 0))
+      (scale (xyz 1 1 1))
+      (rotate (xyz 0 0 0))
+    )
+  )
   (footprint "Mlab_Batery:LTO1865-13_D19.0mm_P7.50mm" (layer "F.Cu")
     (at 129.53 104.102)
@@
   (gr_arc (start 114.554 77.602) (mid 117.482932 70.530932) (end 124.554 67.602) (layer "Edge.Cuts") (width 0.1))
   (gr_line (start 114.554 117.348) (end 175.006 117.348) (layer "Edge.Cuts") (width 0.1))
-  (gr_text "MLAB.CZ\n2022" (at 120.142 92.202 90) (layer "F.SilkS")
+  (gr_text "4XLTO1865V01A\nJACHO" (at 133.35 72.136) (layer "B.SilkS")
+    (effects (font (size 1.5 1.5) (thickness 0.3)) (justify mirror))
+  )
+  (gr_text "MLAB.CZ\n2022" (at 169.291 109.093) (layer "B.SilkS")
+    (effects (font (size 1.5 1.5) (thickness 0.3)) (justify mirror))
+  )
+  (gr_text "MLAB.CZ\n2022" (at 119.38 81.026 90) (layer "F.SilkS")
     (effects (font (size 1.5 1.5) (thickness 0.3)))
   )
-  (gr_text "4XLTO1865V01A\nJACHO" (at 169.926 91.948 90) (layer "F.SilkS")
+  (gr_text "4XLTO1865V01A\nJACHO" (at 170.18 78.994 90) (layer "F.SilkS")
     (effects (font (size 1.5 1.5) (thickness 0.3)))
   )
@@
   (via (at 167.386 115.57) (size 0.9) (drill 0.5) (layers "F.Cu" "B.Cu") (free) (net 3))
   (via (at 122.174 115.57) (size 0.9) (drill 0.5) (layers "F.Cu" "B.Cu") (free) (net 3))
+  (segment (start 144.65 93.472) (end 144.78 93.602) (width 0.5) (layer "F.Cu") (net 4))
+  (segment (start 141.732 93.472) (end 144.65 93.472) (width 0.5) (layer "F.Cu") (net 4))
+  (via (at 141.732 93.472) (size 0.89) (drill 0.5) (layers "F.Cu" "B.Cu") (net 4))
+  (segment (start 130.937 93.472) (end 141.732 93.472) (width 0.5) (layer "B.Cu") (net 4))
+  (segment (start 121.57 102.839) (end 130.937 93.472) (width 0.5) (layer "B.Cu") (net 4))
+  (segment (start 121.57 113.102) (end 121.57 102.839) (width 0.5) (layer "B.Cu") (net 4))
+  (segment (start 141.824 91.602) (end 141.732 91.694) (width 0.5) (layer "F.Cu") (net 5))
+  (segment (start 144.78 91.602) (end 141.824 91.602) (width 0.5) (layer "F.Cu") (net 5))
+  (via (at 141.732 91.694) (size 0.89) (drill 0.5) (layers "F.Cu" "B.Cu") (net 5))
+  (segment (start 130.683 91.694) (end 118.999 103.378) (width 0.5) (layer "B.Cu") (net 5))
+  (segment (start 141.732 91.694) (end 130.683 91.694) (width 0.5) (layer "B.Cu") (net 5))
+  (segment (start 119.03 103.409) (end 119.03 113.102) (width 0.5) (layer "B.Cu") (net 5))
+  (segment (start 118.999 103.378) (end 119.03 103.409) (width 0.5) (layer "B.Cu") (net 5))
   (zone (net 3) (net_name "GND") (layers F&B.Cu) (hatch edge 0.508)
     (connect_pads yes (clearance 0.2))
