File: hw/sch_pcb/4XLTO1865V01A.kicad_sch (KiCad schematic)
At the start: 7 parts, among them J1 HEADER_2x04_PARALLEL, J2 HEADER_2x04_PARALLEL, J3 HEADER_2x04_PARALLEL

Commit message: Edit PCB
Parts:
- added M1, M2: HOLE, Mlab_Mechanical:MountingHole_3mm, symbol MLAB_MECHANICAL:HOLE
- added R1: 10K NTC, Resistor_SMD:R_0805_2012Metric_Pad1.20x1.40mm_HandSolder, symbol LION2CELL01D-rescue:R-RESCUE-LION2CELL01C
Connections:
- net GND: now also M1.1, M2.1; no longer J2.2, J2.3
- new net: J2.2, R1.2
- new net: J2.3, R1.1
Changed lines of the file:
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@@
   (junction (at 186.055 100.965) (diameter 0) (color 0 0 0 0)
   )
-  (junction (at 243.205 20.32) (diameter 0) (color 0 0 0 0)
-  )
-  (junction (at 243.205 22.86) (diameter 0) (color 0 0 0 0)
-  )
   (junction (at 187.96 97.155) (diameter 0) (color 0 0 0 0)
   )
@@
     (stroke (width 0) (type default) (color 0 0 0 0))
   )
-  (wire (pts (xy 243.205 20.32) (xy 243.205 22.86))
-    (stroke (width 0) (type default) (color 0 0 0 0))
-  )
-  (wire (pts (xy 243.205 22.86) (xy 245.11 22.86))
-    (stroke (width 0) (type default) (color 0 0 0 0))
-  )
   (wire (pts (xy 243.205 36.83) (xy 243.205 39.37))
     (stroke (width 0) (type default) (color 0 0 0 0))
@@
     (stroke (width 0) (type default) (color 0 0 0 0))
   )
+  (wire (pts (xy 245.11 20.32) (xy 233.045 20.32))
+    (stroke (width 0) (type default) (color 0 0 0 0))
+  )
   (wire (pts (xy 243.205 25.4) (xy 243.205 27.305))
     (stroke (width 0) (type default) (color 0 0 0 0))
@@
     (stroke (width 0) (type default) (color 0 0 0 0))
   )
-  (wire (pts (xy 243.205 20.32) (xy 245.11 20.32))
-    (stroke (width 0) (type default) (color 0 0 0 0))
-  )
   (wire (pts (xy 243.205 25.4) (xy 245.11 25.4))
     (stroke (width 0) (type default) (color 0 0 0 0))
@@
     (stroke (width 0) (type default) (color 0 0 0 0))
   )
+  (wire (pts (xy 233.045 16.51) (xy 228.6 16.51))
+    (stroke (width 0) (type default) (color 0 0 0 0))
+  )
   (wire (pts (xy 245.11 36.83) (xy 243.205 36.83))
     (stroke (width 0) (type default) (color 0 0 0 0))
@@
     (stroke (width 0) (type default) (color 0 0 0 0))
   )
-  (wire (pts (xy 243.205 22.86) (xy 243.205 25.4))
+  (wire (pts (xy 243.205 17.78) (xy 243.205 25.4))
     (stroke (width 0) (type default) (color 0 0 0 0))
   )
@@
     (stroke (width 0) (type default) (color 0 0 0 0))
   )
-  (wire (pts (xy 243.205 17.78) (xy 243.205 20.32))
+  (wire (pts (xy 23.495 22.225) (xy 27.94 22.225))
+    (stroke (width 0) (type default) (color 0 0 0 0))
+  )
+  (wire (pts (xy 228.6 16.51) (xy 228.6 17.145))
+    (stroke (width 0) (type default) (color 0 0 0 0))
+  )
+  (wire (pts (xy 228.6 29.845) (xy 228.6 30.48))
+    (stroke (width 0) (type default) (color 0 0 0 0))
+  )
+  (wire (pts (xy 228.6 30.48) (xy 233.045 30.48))
     (stroke (width 0) (type default) (color 0 0 0 0))
   )
@@
     (stroke (width 0) (type default) (color 0 0 0 0))
   )
+  (wire (pts (xy 23.495 31.75) (xy 27.94 31.75))
+    (stroke (width 0) (type default) (color 0 0 0 0))
+  )
   (wire (pts (xy 243.205 44.45) (xy 245.11 44.45))
     (stroke (width 0) (type default) (color 0 0 0 0))
@@
     (stroke (width 0) (type default) (color 0 0 0 0))
   )
+  (wire (pts (xy 233.045 20.32) (xy 233.045 16.51))
+    (stroke (width 0) (type default) (color 0 0 0 0))
+  )
   (wire (pts (xy 243.205 39.37) (xy 245.11 39.37))
     (stroke (width 0) (type default) (color 0 0 0 0))
@@
     (stroke (width 0) (type default) (color 0 0 0 0))
   )
+  (wire (pts (xy 233.045 30.48) (xy 233.045 22.86))
+    (stroke (width 0) (type default) (color 0 0 0 0))
+  )
   (wire (pts (xy 243.205 39.37) (xy 243.205 41.91))
     (stroke (width 0) (type default) (color 0 0 0 0))
   )
+  (wire (pts (xy 233.045 22.86) (xy 245.11 22.86))
+    (stroke (width 0) (type default) (color 0 0 0 0))
+  )
   (wire (pts (xy 189.23 95.885) (xy 187.96 95.885))
     (stroke (width 0) (type default) (color 0 0 0 0))
@@
   )
   (wire (pts (xy 187.96 98.425) (xy 189.23 98.425))
+    (stroke (width 0) (type default) (color 0 0 0 0))
+  )
+  (wire (pts (xy 27.94 31.75) (xy 27.94 32.385))
+    (stroke (width 0) (type default) (color 0 0 0 0))
+  )
+  (wire (pts (xy 27.94 22.225) (xy 27.94 22.86))
     (stroke (width 0) (type default) (color 0 0 0 0))
   )
@@
     (effects (font (size 1.524 1.524)) (justify left))
   )
+  (symbol (lib_id "MLAB_MECHANICAL:HOLE") (at 22.225 22.225 0) (unit 1)
+    (in_bom yes) (on_board yes) (fields_autoplaced)
+    (property "Reference" "M1" (id 0) (at 22.225 17.0591 0)
+      (effects (font (size 1.524 1.524)))
+    )
+    (property "Value" "HOLE" (id 1) (at 22.225 20.3381 0)
+      (effects (font (size 1.524 1.524)))
+    )
+    (property "Footprint" "Mlab_Mechanical:MountingHole_3mm" (id 2) (at 22.225 22.225 0)
+      (effects (font (size 1.524 1.524)) hide)
+    )
+    (property "Datasheet" "" (id 3) (at 22.225 22.225 0)
+      (effects (font (size 1.524 1.524)))
+    )
+    (pin "1")
+  )
   (symbol (lib_id "power:GND") (at 243.205 46.355 0) (unit 1)
     (in_bom yes) (on_board yes) (fields_autoplaced)
@@
     (pin "2")
   )
+  (symbol (lib_id "MLAB_MECHANICAL:HOLE") (at 22.225 31.75 0) (unit 1)
+    (in_bom yes) (on_board yes) (fields_autoplaced)
+    (property "Reference" "M2" (id 0) (at 22.225 26.5841 0)
+      (effects (font (size 1.524 1.524)))
+    )
+    (property "Value" "HOLE" (id 1) (at 22.225 29.8631 0)
+      (effects (font (size 1.524 1.524)))
+    )
+    (property "Footprint" "Mlab_Mechanical:MountingHole_3mm" (id 2) (at 22.225 31.75 0)
+      (effects (font (size 1.524 1.524)) hide)
+    )
+    (property "Datasheet" "" (id 3) (at 22.225 31.75 0)
+      (effects (font (size 1.524 1.524)))
+    )
+    (pin "1")
+  )
   (symbol (lib_id "Device:Battery_Cell") (at 151.13 99.06 0) (unit 1)
     (in_bom yes) (on_board yes) (fields_autoplaced)
@@
     (pin "1")
     (pin "2")
+  )
+  (symbol (lib_id "power:GND") (at 27.94 32.385 0) (unit 1)
+    (in_bom yes) (on_board yes) (fields_autoplaced)
+    (property "Reference" "#PWR0103" (id 0) (at 27.94 38.735 0)
+      (effects (font (size 1.27 1.27)) hide)
+    )
+    (property "Value" "GND" (id 1) (at 27.94 36.9475 0))
+    (property "Footprint" "" (id 2) (at 27.94 32.385 0)
+      (effects (font (size 1.27 1.27)) hide)
+    )
+    (property "Datasheet" "" (id 3) (at 27.94 32.385 0)
+      (effects (font (size 1.27 1.27)) hide)
+    )
+    (pin "1")
   )
   (symbol (lib_id "MLAB_HEADER:HEADER_1x04") (at 250.19 21.59 0) (unit 1)
@@
     (pin "4")
   )
+  (symbol (lib_id "LION2CELL01D-rescue:R-RESCUE-LION2CELL01C") (at 228.6 23.495 180) (unit 1)
+    (in_bom yes) (on_board yes)
+    (property "Reference" "R1" (id 0) (at 226.568 23.495 90)
+      (effects (font (size 1.016 1.016)))
+    )
+    (property "Value" "10K NTC" (id 1) (at 228.6 23.495 90)
+      (effects (font (size 1.016 1.016)))
+    )
+    (property "Footprint" "Resistor_SMD:R_0805_2012Metric_Pad1.20x1.40mm_HandSolder" (id 2) (at 230.378 23.495 90)
+      (effects (font (size 0.762 0.762)) hide)
+    )
+    (property "Datasheet" "" (id 3) (at 228.6 23.495 0)
+      (effects (font (size 0.762 0.762)))
+    )
+    (pin "1")
+    (pin "2")
+  )
   (symbol (lib_id "MLAB_HEADER:HEADER_1x04") (at 194.31 97.155 0) (unit 1)
     (in_bom yes) (on_board yes) (fields_autoplaced)
@@
     (pin "3")
     (pin "4")
+  )
+  (symbol (lib_id "power:GND") (at 27.94 22.86 0) (unit 1)
+    (in_bom yes) (on_board yes) (fields_autoplaced)
+    (property "Reference" "#PWR0104" (id 0) (at 27.94 29.21 0)
+      (effects (font (size 1.27 1.27)) hide)
+    )
+    (property "Value" "GND" (id 1) (at 27.94 27.4225 0))
+    (property "Footprint" "" (id 2) (at 27.94 22.86 0)
+      (effects (font (size 1.27 1.27)) hide)
+    )
+    (property "Datasheet" "" (id 3) (at 27.94 22.86 0)
+      (effects (font (size 1.27 1.27)) hide)
+    )
+    (pin "1")
   )
   (symbol (lib_id "Device:Battery_Cell") (at 112.395 99.06 0) (unit 1)
@@
       (reference "#PWR0102") (unit 1) (value "GND") (footprint "")
     )
+    (path "/7b98f520-9064-4449-b7d1-5fd5af720bc5"
+      (reference "#PWR0103") (unit 1) (value "GND") (footprint "")
+    )
+    (path "/ec583818-8f10-4faf-b5e2-d073ba38f33b"
+      (reference "#PWR0104") (unit 1) (value "GND") (footprint "")
+    )
     (path "/20d20a6c-03cf-4a4c-8a77-7b10171706e4"
       (reference "BT1") (unit 1) (value "LTO1865-13") (footprint "Mlab_Batery:LTO1865-13_D19.0mm_P7.50mm")
@@
       (reference "J3") (unit 1) (value "HEADER_2x04_PARALLEL") (footprint "Mlab_Pin_Headers:Angled_1x04")
     )
-  )
+    (path "/01473b40-a501-4b7d-9200-f7912f5aad08"
+      (reference "M1") (unit 1) (value "HOLE") (footprint "Mlab_Mechanical:MountingHole_3mm")
+    )
+    (path "/3891a704-a6c9-482e-81b2-d42bd6e42e53"
+      (reference "M2") (unit 1) (value "HOLE") (footprint "Mlab_Mechanical:MountingHole_3mm")
+    )
+    (path "/84282cc7-416d-48c2-ae9f-c0149b35065e"
+      (reference "R1") (unit 1) (value "10K NTC") (footprint "Resistor_SMD:R_0805_2012Metric_Pad1.20x1.40mm_HandSolder")
+    )
+  )
